Commit message: Update follower platooning reverse turn support

File: turtlebot3_manipulation/turtlebot3_manipulation_description/urdf/turtlebot3_platooning.urdf (robot description, URDF)
Before this commit: robot turtlebot3_platooning, 10 links, 9 joints
Links:
- added link cargo_deck_link, mass 0.050; collision box size=0.180 0.160 0.012; visual box size=0.180 0.160 0.012
Joints:
- added joint cargo_deck_joint: type fixed, parent base_link, child cargo_deck_link, origin xyz=-0.045 0 0.105 rpy=0 0 0

File: turtlebot3_manipulation/turtlebot3_manipulation_description/xacro/turtlebot3_platooning.xacro (robot description, xacro)
@@ -140,4 +140,31 @@
   </joint>
   <link name="${prefix}imu_link"/>
+  <joint name="${prefix}cargo_deck_joint" type="fixed">
+    <parent link="${prefix}base_link"/>
+    <child link="${prefix}cargo_deck_link"/>
+    <origin xyz="-0.045 0 0.105" rpy="0 0 0"/>
+  </joint>
+  <link name="${prefix}cargo_deck_link">
+    <visual>
+      <origin xyz="0 0 0" rpy="0 0 0"/>
+      <geometry>
+        <box size="0.180 0.160 0.012"/>
+      </geometry>
+      <material name="dark"/>
+    </visual>
+    <collision>
+      <origin xyz="0 0 0" rpy="0 0 0"/>
+      <geometry>
+        <box size="0.180 0.160 0.012"/>
+      </geometry>
+    </collision>
+    <inertial>
+      <origin xyz="0 0 0" />
+      <mass value="0.050" />
+      <inertia ixx="1.117e-04" ixy="0.0" ixz="0.0"
+               iyy="1.620e-04" iyz="0.0"
+               izz="2.417e-04" />
+    </inertial>
+  </link>
   <joint name="${prefix}camera_joint" type="fixed">
     <parent link="${prefix}base_link"/>
